File: END67.kicad_pcb (KiCad board)
At the start: 2 copper layers, 150 parts, among them SW1 SW_Push, U1 ATmega32U4-AU, Y1 16MHz

Commit message: Finished First Prototype
Parts:
- C7: value 0.1uF -> 10uF
Changed lines of the file:
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@@
       (effects (font (size 1 1) (thickness 0.15)))
     )
-    (fp_text value 0.1uF (at 0 1.65) (layer F.Fab)
+    (fp_text value 10uF (at 0 1.65) (layer F.Fab)
       (effects (font (size 1 1) (thickness 0.15)))
     )
