File: END67vOut.kicad_pcb (KiCad board)
At the start: 2 copper layers, 150 parts, among them SW1 SW_Push, U1 ATmega32U4-AU, Y1 16MHz

Commit message: Finished First Prototype
Parts:
- C1, C2, C3, C4, C5, C6, D0, D0A1, D0B1, D0C1, D0D1, D0E1, D1, D10, D11, D12, D13, D14, D15, D16, D17, D18, D19, D1A1, D1B1, D1C1, D1D1, D1E1, D2, D20, D21, D22, D23, D24, D25, D26, D27, D28, D29, D2A1, D2B1, D2C1, D2D1, D2E1, D3, D30, D31, D32, D33, D34, D35, D36, D37, D38, D39, D3A1, D3B1, D3C1, D3D1, D4, D41, D42, D46, D4A1, D4B1, D4C1, D4D1, D4E1, D5, D6, D7, D8, D9, F1, R1, R2, R3, R4, SW1, U1, USB1, Y1: moved to B.Cu
- C7: value 0.1uF -> 10uF; moved to B.Cu
- moved SW1 316.3 mm to (362.6, 95.7)
- moved F1 304.2 mm to (338.9, 95.9), turned to 270 degrees
- moved Y1 282.0 mm to (360.5, 135.6), turned to 180 degrees
- moved C5 272.9 mm to (370.1, 142.5), turned to 90 degrees
- moved R3 271.1 mm to (344.4, 95.9), turned to 90 degrees
- moved C1 266.9 mm to (365.4, 135.8), turned to 90 degrees
- moved C6 264.5 mm to (365.5, 156.1), turned to 180 degrees
- moved C7 260.9 mm to (356.1, 156.1)
- moved C4 258.2 mm to (352.7, 140.0), turned to 90 degrees
- moved C2 253.2 mm to (355.6, 135.8), turned to 270 degrees
- moved R4 248.5 mm to (369.8, 152.3), turned to 90 degrees
- moved C3 245.2 mm to (351.4, 147.6), turned to 180 degrees
- moved D4E1 210.9 mm to (262.7, 97.6), turned to 270 degrees
- moved D4D1 209.0 mm to (250.8, 97.6), turned to 270 degrees
- moved R2 208.7 mm to (346.8, 95.9), turned to 90 degrees
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Other:
- board outline added: 343.7 x 122.2 mm
