File: END67vOutFirst.sch (KiCad schematic (older format))
At the start: 150 parts, among them SW1 SW_Push, U1 ATmega32U4-AU, Y1 16MHz

Commit message: Finished First Prototype
Connections:
- net COL0: now also U1.25 (PD4); no longer U1.8 (PB0)
- net COL1: now also U1.26 (PD6); no longer U1.9 (PB1)
- net COL10: now also U1.11 (PB3); no longer U1.25 (PD4)
- net COL11: now also U1.18 (PD0); no longer U1.21 (PD3)
- net COL12: now also U1.19 (PD1); no longer U1.20 (PD2)
- net COL13: now also U1.20 (PD2); no longer U1.19 (PD1)
- net COL14: now also U1.21 (PD3); no longer U1.18 (PD0)
- net COL2: now also U1.27 (PD7); no longer U1.10 (PB2)
- net COL3: now also U1.28 (PB4); no longer U1.11 (PB3)
- net COL4: now also U1.29 (PB5); no longer U1.31 (PC6)
- net COL6: now also U1.31 (PC6); no longer U1.29 (PB5)
- net COL7: now also U1.8 (PB0); no longer U1.28 (PB4)
- net COL8: now also U1.9 (PB1); no longer U1.27 (PD7)
- net COL9: now also U1.10 (PB2); no longer U1.26 (PD6)
- no-connect marks 8 -> 13
Changed lines of the file:
@@
 EESchema Schematic File Version 4
-LIBS:END67-cache
 EELAYER 30 0
 EELAYER END
@@
 Wire Wire Line
 	3350 3700 3450 3700
+Text GLabel 3450 2800 2    50   Input ~ 0
+COL14
+Text GLabel 3450 2700 2    50   Input ~ 0
+COL13
+Text GLabel 3450 2600 2    50   Input ~ 0
+COL12
 Text GLabel 3450 2500 2    50   Input ~ 0
-COL14
-Text GLabel 3450 2600 2    50   Input ~ 0
-COL13
-Text GLabel 3450 2700 2    50   Input ~ 0
-COL12
-Text GLabel 3450 2800 2    50   Input ~ 0
 COL11
-Text GLabel 3450 2900 2    50   Input ~ 0
-COL10
-Text GLabel 3450 3100 2    50   Input ~ 0
-COL9
-Text GLabel 3450 3200 2    50   Input ~ 0
+Text GLabel 3450 1400 2    50   Input ~ 0
 COL8
-Text GLabel 3450 1700 2    50   Input ~ 0
+Text GLabel 3450 1300 2    50   Input ~ 0
 COL7
-Text GLabel 3450 1800 2    50   Input ~ 0
+Text GLabel 3450 2200 2    50   Input ~ 0
 COL6
 Text GLabel 3450 1900 2    50   Input ~ 0
 COL5
-Text GLabel 3450 2200 2    50   Input ~ 0
+Text GLabel 3450 1800 2    50   Input ~ 0
 COL4
-Text GLabel 3450 1600 2    50   Input ~ 0
+Text GLabel 3450 1700 2    50   Input ~ 0
 COL3
-Text GLabel 3450 1500 2    50   Input ~ 0
+Text GLabel 3450 3200 2    50   Input ~ 0
 COL2
-Text GLabel 3450 1400 2    50   Input ~ 0
+Text GLabel 3450 3100 2    50   Input ~ 0
 COL1
-Text GLabel 3450 1300 2    50   Input ~ 0
-COL0
 Wire Wire Line
 	3350 3200 3450 3200
@@
 	1    0    0    -1
 $EndComp
+Text GLabel 3450 1500 2    50   Input ~ 0
+COL9
+Text GLabel 3450 1600 2    50   Input ~ 0
+COL10
+Text GLabel 3450 2900 2    50   Input ~ 0
+COL0
+NoConn ~ 3350 3500
+NoConn ~ 3350 4200
+NoConn ~ 3350 2300
+NoConn ~ 3350 2000
+NoConn ~ 2150 1900
 $EndSCHEMATC
